File: Keithley1950.sch (KiCad schematic (older format))
At the start: 89 parts, among them J1 Conn_01x14, J2 Conn_01x03, J3 Conn_01x02, K1 Relay_SP2P, K2 Relay_SP2P, K3 Relay_SP3P, K4 Relay_SP2P, K5 Relay_SP2P, K6 Relay_SP3P, K7 Relay_SP3P, Q1 MMBFJ111, Q2 MMBFJ111, Q3 MMBFJ111, Q4 MMBFJ111, Q5 MMBT3906, Q6 MMBT3906, Q7 MMBFJ111, Q8 MMBT3906, U1 TL082, U2 LM339, U3 74LS138, U4 AD8436, U5 ULN2003, U6 74HC4094, U7 TL082

Commit message: Add constantan spiral model
Parts:
- U2: footprint Package_SO:SOIC-8_3.9x4.9mm_P1.27mm -> Package_SO:SOIC-14_3.9x8.7mm_P1.27mm
Changed lines of the file:
@@
 F 0 "U2" H 7600 1800 50  0000 C CNN
 F 1 "LM339" H 7650 1700 50  0000 C CNN
-F 2 "Package_SO:SOIC-8_3.9x4.9mm_P1.27mm" H 7450 1550 50  0001 C CNN
+F 2 "Package_SO:SOIC-14_3.9x8.7mm_P1.27mm" H 7450 1550 50  0001 C CNN
 F 3 "http://www.ti.com/lit/ds/symlink/lm339.pdf" H 7550 1650 50  0001 C CNN
 	1    7500 1450
@@
 F 0 "U2" H 7500 2175 50  0000 C CNN
 F 1 "LM339" H 7500 2176 50  0001 C CNN
-F 2 "Package_SO:SOIC-8_3.9x4.9mm_P1.27mm" H 7450 2000 50  0001 C CNN
+F 2 "Package_SO:SOIC-14_3.9x8.7mm_P1.27mm" H 7450 2000 50  0001 C CNN
 F 3 "http://www.ti.com/lit/ds/symlink/lm339.pdf" H 7550 2100 50  0001 C CNN
 	2    7500 1900
@@
 F 0 "U2" H 7500 2625 50  0000 C CNN
 F 1 "LM339" H 7500 2626 50  0001 C CNN
-F 2 "Package_SO:SOIC-8_3.9x4.9mm_P1.27mm" H 7450 2450 50  0001 C CNN
+F 2 "Package_SO:SOIC-14_3.9x8.7mm_P1.27mm" H 7450 2450 50  0001 C CNN
 F 3 "http://www.ti.com/lit/ds/symlink/lm339.pdf" H 7550 2550 50  0001 C CNN
 	3    7500 2350
@@
 F 0 "U2" H 7500 3075 50  0000 C CNN
 F 1 "LM339" H 7500 3076 50  0001 C CNN
-F 2 "Package_SO:SOIC-8_3.9x4.9mm_P1.27mm" H 7450 2900 50  0001 C CNN
+F 2 "Package_SO:SOIC-14_3.9x8.7mm_P1.27mm" H 7450 2900 50  0001 C CNN
 F 3 "http://www.ti.com/lit/ds/symlink/lm339.pdf" H 7550 3000 50  0001 C CNN
 	4    7500 2800
@@
 F 0 "U2" H 7658 1450 50  0001 L CNN
 F 1 "LM339" H 7658 1405 50  0001 L CNN
-F 2 "Package_SO:SOIC-8_3.9x4.9mm_P1.27mm" H 7650 1550 50  0001 C CNN
+F 2 "Package_SO:SOIC-14_3.9x8.7mm_P1.27mm" H 7650 1550 50  0001 C CNN
 F 3 "http://www.ti.com/lit/ds/symlink/lm339.pdf" H 7750 1650 50  0001 C CNN
 	5    7700 1450
@@
 F 0 "U2" H 7700 3000 50  0001 L CNN
 F 1 "LM339" H 7700 2600 50  0001 L CNN
-F 2 "Package_SO:SOIC-8_3.9x4.9mm_P1.27mm" H 7650 2900 50  0001 C CNN
+F 2 "Package_SO:SOIC-14_3.9x8.7mm_P1.27mm" H 7650 2900 50  0001 C CNN
 F 3 "http://www.ti.com/lit/ds/symlink/lm339.pdf" H 7750 3000 50  0001 C CNN
 	6    7700 2800

Commit message: Initial placement on pcb
Parts:
- added H1, H2, H3: MountingHole_Pad, MountingHole:MountingHole_3.2mm_M3_Pad_Via, symbol Mechanical:MountingHole_Pad
- D1, D2, D3, D4, D5, D6, D7: footprint Diode_SMD:D_SMC -> Diode_SMD:D_SMB-SMC_Universal_Handsoldering
- J1: footprint Connector_IDC:IDC-Header_2x07_P2.54mm_Vertical -> Package_DIP:DIP-14_W7.62mm_Socket_LongPads
Connections:
- no-connect marks 7 -> 10
Changed lines of the file:
@@
 F 0 "J1" H 10918 2125 50  0000 C CNN
 F 1 "Conn_01x14" H 10918 2216 50  0000 C CNN
-F 2 "Connector_IDC:IDC-Header_2x07_P2.54mm_Vertical" H 11000 3050 50  0001 C CNN
+F 2 "Package_DIP:DIP-14_W7.62mm_Socket_LongPads" H 11000 3050 50  0001 C CNN
 F 3 "~" H 11000 3050 50  0001 C CNN
 	1    11000 3050
@@
 F 0 "D7" H 2800 7000 50  0000 C CNN
 F 1 "S3M" H 3000 7000 50  0000 C CNN
-F 2 "Diode_SMD:D_SMC" V 2900 7100 50  0001 C CNN
+F 2 "Diode_SMD:D_SMB-SMC_Universal_Handsoldering" V 2900 7100 50  0001 C CNN
 F 3 "~" V 2900 7100 50  0001 C CNN
 	1    2900 7100
@@
 F 0 "D6" H 3000 6850 50  0000 C CNN
 F 1 "S3M" H 2800 6850 50  0000 C CNN
-F 2 "Diode_SMD:D_SMC" V 2900 6950 50  0001 C CNN
+F 2 "Diode_SMD:D_SMB-SMC_Universal_Handsoldering" V 2900 6950 50  0001 C CNN
 F 3 "~" V 2900 6950 50  0001 C CNN
 	1    2900 6950
@@
 F 0 "D3" H 1900 4150 50  0000 C CNN
 F 1 "S3M" H 1650 4150 50  0000 C CNN
-F 2 "Diode_SMD:D_SMC" V 1800 4200 50  0001 C CNN
+F 2 "Diode_SMD:D_SMB-SMC_Universal_Handsoldering" V 1800 4200 50  0001 C CNN
 F 3 "~" V 1800 4200 50  0001 C CNN
 	1    1800 4200
@@
 F 0 "D4" H 1550 4450 50  0000 C CNN
 F 1 "S3M" H 1700 4450 50  0000 C CNN
-F 2 "Diode_SMD:D_SMC" V 1650 4350 50  0001 C CNN
+F 2 "Diode_SMD:D_SMB-SMC_Universal_Handsoldering" V 1650 4350 50  0001 C CNN
 F 3 "~" V 1650 4350 50  0001 C CNN
 	1    1650 4350
@@
 F 0 "D5" H 1900 4450 50  0000 C CNN
 F 1 "S3M" H 2050 4450 50  0000 C CNN
-F 2 "Diode_SMD:D_SMC" V 1950 4350 50  0001 C CNN
+F 2 "Diode_SMD:D_SMB-SMC_Universal_Handsoldering" V 1950 4350 50  0001 C CNN
 F 3 "~" V 1950 4350 50  0001 C CNN
 	1    1950 4350
@@
 F 0 "D2" H 1950 4255 50  0000 C CNN
 F 1 "S3M" H 1950 4164 50  0000 C CNN
-F 2 "Diode_SMD:D_SMC" V 1950 4050 50  0001 C CNN
+F 2 "Diode_SMD:D_SMB-SMC_Universal_Handsoldering" V 1950 4050 50  0001 C CNN
 F 3 "~" V 1950 4050 50  0001 C CNN
 	1    1950 4050
@@
 F 0 "D1" H 1650 4255 50  0000 C CNN
 F 1 "S3M" H 1650 4164 50  0000 C CNN
-F 2 "Diode_SMD:D_SMC" V 1650 4050 50  0001 C CNN
+F 2 "Diode_SMD:D_SMB-SMC_Universal_Handsoldering" V 1650 4050 50  0001 C CNN
 F 3 "~" V 1650 4050 50  0001 C CNN
 	1    1650 4050
@@
 Wire Wire Line
 	1200 5750 1200 5700
+$Comp
+L Mechanical:MountingHole_Pad H1
+U 1 1 5D327519
+P 950 7400
+F 0 "H1" H 1050 7449 50  0000 L CNN
+F 1 "MountingHole_Pad" H 600 7600 50  0000 L CNN
+F 2 "MountingHole:MountingHole_3.2mm_M3_Pad_Via" H 950 7400 50  0001 C CNN
+F 3 "~" H 950 7400 50  0001 C CNN
+	1    950  7400
+	1    0    0    -1
+$EndComp
+$Comp
+L Mechanical:MountingHole_Pad H2
+U 1 1 5D327849
+P 1300 7400
+F 0 "H2" H 1400 7449 50  0000 L CNN
+F 1 "MountingHole_Pad" H 950 7150 50  0000 L CNN
+F 2 "MountingHole:MountingHole_3.2mm_M3_Pad_Via" H 1300 7400 50  0001 C CNN
+F 3 "~" H 1300 7400 50  0001 C CNN
+	1    1300 7400
+	1    0    0    -1
+$EndComp
+$Comp
+L Mechanical:MountingHole_Pad H3
+U 1 1 5D327A53
+P 1650 7400
+F 0 "H3" H 1750 7449 50  0000 L CNN
+F 1 "MountingHole_Pad" H 1400 7600 50  0000 L CNN
+F 2 "MountingHole:MountingHole_3.2mm_M3_Pad_Via" H 1650 7400 50  0001 C CNN
+F 3 "~" H 1650 7400 50  0001 C CNN
+	1    1650 7400
+	1    0    0    -1
+$EndComp
+NoConn ~ 950  7500
+NoConn ~ 1300 7500
+NoConn ~ 1650 7500
 $EndSCHEMATC
