File: Keithley1950.sch (KiCad schematic (older format))
At the start: 92 parts, among them J1 Conn_01x14, J2 Conn_01x03, J3 Conn_01x02, K1 Relay_SP2P, K2 Relay_SP2P, K3 Relay_SP3P, K4 Relay_SP2P, K5 Relay_SP2P, K6 Relay_SP3P, K7 Relay_SP3P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

Commit message: Optimized placement
Parts:
- D1, D2, D3, D4, D5, D6, D7: footprint Diode_SMD:D_SMB-SMC_Universal_Handsoldering -> Diode_SMD:D_SMB

Commit message: More optimizations
Parts:
- C12: footprint Capacitor_SMD:C_0603_1608Metric -> Capacitor_SMD:C_0805_2012Metric
Changed lines of the file:
@@
 F 0 "C12" H 4042 4796 50  0000 L CNN
 F 1 "3.3uF" H 4042 4705 50  0000 L CNN
-F 2 "Capacitor_SMD:C_0603_1608Metric" H 3950 4750 50  0001 C CNN
+F 2 "Capacitor_SMD:C_0805_2012Metric" H 3950 4750 50  0001 C CNN
 F 3 "~" H 3950 4750 50  0001 C CNN
 	1    3950 4750
